Commit message: v0.1

File: urdf/differential_robot.urdf.xacro (robot description, xacro)
@@ -4,5 +4,5 @@
   <xacro:property name="wheel_radius" value="0.065"/>
   <xacro:property name="wheel_separation" value="0.5"/>
-  <!-- Link principal -->
+  <!-- Link principal (chasis en gris) -->
   <link name="base_link">
     <inertial>
@@ -11,24 +11,21 @@
       <inertia ixx="0.1" ixy="0.0" ixz="0.0" iyy="0.1" iyz="0.0" izz="0.1"/>
     </inertial>
-        <visual>
-        <!-- ajusta origen si tu STL no está centrado -->
-        <origin xyz="0 0 0" rpy="1.57 0 1.57"/>
-        <geometry>
-        <mesh
-            filename="package://robot_description/meshes/base_link.stl"
-            scale="0.003 0.003 0.003"/>
-        </geometry>
-        <material name="blue"/>
+    <visual>
+      <origin xyz="0 0 0" rpy="1.57 0 1.57"/>
+      <geometry>
+        <mesh filename="package://robot_description/meshes/base_link.stl" scale="0.003 0.003 0.003"/>
+      </geometry>
+      <material name="gray">
+        <color rgba="0.5 0.5 0.5 1"/>
+      </material>
     </visual>
     <collision>
-        <origin xyz="0 0 0" rpy="1.57 0 1.57"/>
-        <geometry>
-        <mesh
-            filename="package://robot_description/meshes/base_link.stl"
-            scale="0.003 0.003 0.003"/>
-        </geometry>
+      <origin xyz="0 0 0" rpy="1.57 0 1.57"/>
+      <geometry>
+        <mesh filename="package://robot_description/meshes/base_link.stl" scale="0.003 0.003 0.003"/>
+      </geometry>
     </collision>
   </link>
-  <!-- Rueda izquierda -->
+  <!-- Ruedas motrices (en negro) -->
   <link name="wheel_left_link">
     <inertial>
@@ -42,5 +39,7 @@
         <cylinder length="0.02" radius="${wheel_radius}"/>
       </geometry>
-      <material name="black"/>
+      <material name="black">
+        <color rgba="0 0 0 1"/>
+      </material>
     </visual>
     <collision>
@@ -51,5 +50,4 @@
     </collision>
   </link>
-  <!-- Rueda derecha -->
   <link name="wheel_right_link">
     <inertial>
@@ -63,5 +61,7 @@
         <cylinder length="0.02" radius="${wheel_radius}"/>
       </geometry>
-      <material name="black"/>
+      <material name="black">
+        <color rgba="0 0 0 1"/>
+      </material>
     </visual>
     <collision>
@@ -72,6 +72,22 @@
     </collision>
   </link>
-  <!-- Rueda loca (caster) -->
-  <link name="caster_link">
+  <!-- Caster de bola (en negro) -->
+  <!-- 1) Montaje fijo -->
+  <link name="caster_mount_link"/>
+  <joint name="caster_mount_joint" type="fixed">
+    <parent link="base_link"/>
+    <child link="caster_mount_link"/>
+    <origin xyz="-0.2 0 -0.0125" rpy="0 0 0"/>
+  </joint>
+  <!-- 2) Eje de rotación roll (X) -->
+  <link name="caster_roll_link"/>
+  <joint name="caster_roll_joint" type="continuous">
+    <parent link="caster_mount_link"/>
+    <child link="caster_roll_link"/>
+    <origin xyz="0 0 0" rpy="0 0 0"/>
+    <axis xyz="1 0 0"/>
+  </joint>
+  <!-- 3) Eje de rotación pitch (Y) con la bola -->
+  <link name="caster_ball_link">
     <inertial>
       <origin xyz="0 0 0" rpy="0 0 0"/>
@@ -80,12 +96,14 @@
     </inertial>
     <visual>
-      <origin xyz="0 0 -0.1" rpy="0 0 0"/>
+      <origin xyz="0 0 0" rpy="0 0 0"/>
       <geometry>
         <sphere radius="0.0125"/>
       </geometry>
-      <material name="grey"/>
+      <material name="black">
+        <color rgba="0 0 0 1"/>
+      </material>
     </visual>
     <collision>
-      <origin xyz="0 0 -0.1" rpy="0 0 0"/>
+      <origin xyz="0 0 0" rpy="0 0 0"/>
       <geometry>
         <sphere radius="0.0125"/>
@@ -93,5 +111,11 @@
     </collision>
   </link>
-  <!-- Uniones de las ruedas al chasis -->
+  <joint name="caster_pitch_joint" type="continuous">
+    <parent link="caster_roll_link"/>
+    <child link="caster_ball_link"/>
+    <origin xyz="0 0 0" rpy="0 0 0"/>
+    <axis xyz="0 1 0"/>
+  </joint>
+  <!-- Joints de ruedas motrices -->
   <joint name="joint_wheel_left" type="continuous">
     <parent link="base_link"/>
@@ -105,9 +129,4 @@
     <origin xyz="0 ${wheel_separation/2} 0" rpy="0 0 0"/>
     <axis xyz="0 1 0"/>
-  </joint>
-  <joint name="joint_caster" type="fixed">
-    <parent link="base_link"/>
-    <child link="caster_link"/>
-    <origin xyz="-0.2 0 0" rpy="0 0 0"/>
   </joint>
   <!-- Transmissions -->

Commit message: v0.2

File: urdf/differential_robot.urdf.xacro (robot description, xacro)
@@ -2,6 +2,6 @@
 <robot name="differential_robot" xmlns:xacro="http://www.ros.org/wiki/xacro">
   <!-- Parámetros básicos -->
-  <xacro:property name="wheel_radius" value="0.065"/>
-  <xacro:property name="wheel_separation" value="0.5"/>
+  <xacro:property name="wheel_radius" value="0.0325"/>
+  <xacro:property name="wheel_separation" value="0.095"/>
   <!-- Link principal (chasis en gris) -->
   <link name="base_link">
@@ -14,5 +14,5 @@
       <origin xyz="0 0 0" rpy="1.57 0 1.57"/>
       <geometry>
-        <mesh filename="package://robot_description/meshes/base_link.stl" scale="0.003 0.003 0.003"/>
+        <mesh filename="package://robot_description/meshes/base_link.stl" scale="0.0008 0.0008 0.0008"/>
       </geometry>
       <material name="gray">
@@ -23,5 +23,5 @@
       <origin xyz="0 0 0" rpy="1.57 0 1.57"/>
       <geometry>
-        <mesh filename="package://robot_description/meshes/base_link.stl" scale="0.003 0.003 0.003"/>
+        <mesh filename="package://robot_description/meshes/base_link.stl" scale="0.0008 0.0008 0.0008"/>
       </geometry>
     </collision>
@@ -78,5 +78,5 @@
     <parent link="base_link"/>
     <child link="caster_mount_link"/>
-    <origin xyz="-0.2 0 -0.0125" rpy="0 0 0"/>
+    <origin xyz="-0.035 0 -0.035" rpy="0 0 0"/>
   </joint>
   <!-- 2) Eje de rotación roll (X) -->
@@ -121,5 +121,5 @@
     <parent link="base_link"/>
     <child link="wheel_left_link"/>
-    <origin xyz="0 ${-wheel_separation/2} 0" rpy="0 0 0"/>
+    <origin xyz="0.025 ${-wheel_separation/2} -0.01" rpy="0 0 0"/>
     <axis xyz="0 1 0"/>
   </joint>
@@ -127,5 +127,5 @@
     <parent link="base_link"/>
     <child link="wheel_right_link"/>
-    <origin xyz="0 ${wheel_separation/2} 0" rpy="0 0 0"/>
+    <origin xyz="0.025 ${wheel_separation/2} -0.01" rpy="0 0 0"/>
     <axis xyz="0 1 0"/>
   </joint>

Commit message: v0.5 quito stl y pongo box

File: urdf/differential_robot.urdf.xacro (robot description, xacro)
@@ -12,7 +12,7 @@
     </inertial>
     <visual>
-      <origin xyz="0 0 0" rpy="1.57 0 1.57"/>
+      <origin xyz="0 0 0" rpy="0 0 0"/>
       <geometry>
-        <mesh filename="package://robot_description/meshes/base_link.stl" scale="0.0008 0.0008 0.0008"/>
+        <box size="0.15 0.12 0.05"/>
       </geometry>
       <material name="gray">
@@ -21,7 +21,7 @@
     </visual>
     <collision>
-      <origin xyz="0 0 0" rpy="1.57 0 1.57"/>
+      <origin xyz="0 0 0" rpy="0 0 0"/>
       <geometry>
-        <mesh filename="package://robot_description/meshes/base_link.stl" scale="0.0008 0.0008 0.0008"/>
+        <box size="0.15 0.12 0.05"/>
       </geometry>
     </collision>

Commit message: v0.7 gazebo

File: urdf/differential_robot.urdf.xacro (robot description, xacro)
@@ -74,5 +74,26 @@
   <!-- Caster de bola (en negro) -->
   <!-- 1) Montaje fijo -->
-  <link name="caster_mount_link"/>
+  <link name="caster_mount_link">
+    <inertial>
+      <origin xyz="0 0 0" rpy="0 0 0"/>
+      <mass value="0.1"/>
+      <inertia ixx="0.0001" ixy="0.0" ixz="0.0" iyy="0.0001" iyz="0.0" izz="0.0001"/>
+    </inertial>
+    <visual>
+      <origin xyz="0 0 0" rpy="0 0 0"/>
+      <geometry>
+        <cylinder length="0.02" radius="0.01"/>
+      </geometry>
+      <material name="black">
+        <color rgba="0 0 0 1"/>
+      </material>
+    </visual>
+    <collision>
+      <origin xyz="0 0 0" rpy="0 0 0"/>
+      <geometry>
+        <cylinder length="0.02" radius="0.01"/>
+      </geometry>
+    </collision>
+  </link>
   <joint name="caster_mount_joint" type="fixed">
     <parent link="base_link"/>
@@ -81,5 +102,26 @@
   </joint>
   <!-- 2) Eje de rotación roll (X) -->
-  <link name="caster_roll_link"/>
+  <link name="caster_roll_link">
+    <inertial>
+      <origin xyz="0 0 0" rpy="0 0 0"/>
+      <mass value="0.1"/>
+      <inertia ixx="0.0001" ixy="0.0" ixz="0.0" iyy="0.0001" iyz="0.0" izz="0.0001"/>
+    </inertial>
+    <visual>
+      <origin xyz="0 0 0" rpy="0 0 0"/>
+      <geometry>
+        <cylinder length="0.02" radius="0.005"/>
+      </geometry>
+      <material name="black">
+        <color rgba="0 0 0 1"/>
+      </material>
+    </visual>
+    <collision>
+      <origin xyz="0 0 0" rpy="0 0 0"/>
+      <geometry>
+        <cylinder length="0.02" radius="0.005"/>
+      </geometry>
+    </collision>
+  </link>
   <joint name="caster_roll_joint" type="continuous">
     <parent link="caster_mount_link"/>

Commit message: colores Gazebo

File: urdf/differential_robot.urdf.xacro (robot description, xacro)
@@ -183,3 +183,21 @@
     <actuator name="motor_right"/>
   </transmission>
+  <gazebo reference="base_link">
+    <material>Gazebo/White</material>
+  </gazebo>
+  <gazebo reference="wheel_left_link">
+    <material>Gazebo/Black</material>
+  </gazebo>
+  <gazebo reference="wheel_right_link">
+    <material>Gazebo/Black</material>
+  </gazebo>
+  <gazebo reference="caster_mount_link">
+    <material>Gazebo/Blue</material>
+  </gazebo>
+  <gazebo reference="caster_roll_link">
+    <material>Gazebo/Blue</material>
+  </gazebo>
+  <gazebo reference="caster_ball_link">
+    <material>Gazebo/Blue</material>
+  </gazebo>
 </robot>

Commit message: v0.8gazebo plugin

File: urdf/differential_robot.urdf.xacro (robot description, xacro)
@@ -8,5 +8,5 @@
     <inertial>
       <origin xyz="0 0 0" rpy="0 0 0"/>
-      <mass value="5.0"/>
+      <mass value="1.0"/>
       <inertia ixx="0.1" ixy="0.0" ixz="0.0" iyy="0.1" iyz="0.0" izz="0.1"/>
     </inertial>
@@ -31,5 +31,5 @@
     <inertial>
       <origin xyz="0 0 0" rpy="0 0 0"/>
-      <mass value="1.0"/>
+      <mass value="0.05"/>
       <inertia ixx="0.01" ixy="0.0" ixz="0.0" iyy="0.01" iyz="0.0" izz="0.01"/>
     </inertial>
@@ -53,5 +53,5 @@
     <inertial>
       <origin xyz="0 0 0" rpy="0 0 0"/>
-      <mass value="1.0"/>
+      <mass value="0.05"/>
       <inertia ixx="0.01" ixy="0.0" ixz="0.0" iyy="0.01" iyz="0.0" izz="0.01"/>
     </inertial>
@@ -77,5 +77,5 @@
     <inertial>
       <origin xyz="0 0 0" rpy="0 0 0"/>
-      <mass value="0.1"/>
+      <mass value="0.05"/>
       <inertia ixx="0.0001" ixy="0.0" ixz="0.0" iyy="0.0001" iyz="0.0" izz="0.0001"/>
     </inertial>

Commit message: v1

File: urdf/differential_robot.urdf.xacro (robot description, xacro)
@@ -124,9 +124,11 @@
     </collision>
   </link>
-  <joint name="caster_roll_joint" type="continuous">
+  <joint name="caster_roll_joint" type="revolute">
     <parent link="caster_mount_link"/>
     <child link="caster_roll_link"/>
     <origin xyz="0 0 0" rpy="0 0 0"/>
     <axis xyz="1 0 0"/>
+    <limit lower="-3.14159" upper="3.14159" effort="0" velocity="0"/>
+    <dynamics damping="0.1" friction="0.1"/>
   </joint>
   <!-- 3) Eje de rotación pitch (Y) con la bola -->
@@ -153,9 +155,11 @@
     </collision>
   </link>
-  <joint name="caster_pitch_joint" type="continuous">
+  <joint name="caster_pitch_joint" type="revolute">
     <parent link="caster_roll_link"/>
     <child link="caster_ball_link"/>
     <origin xyz="0 0 0" rpy="0 0 0"/>
     <axis xyz="0 1 0"/>
+    <limit lower="-3.14159" upper="3.14159" effort="0" velocity="0"/>
+    <dynamics damping="0.1" friction="0.1"/>
   </joint>
   <!-- Joints de ruedas motrices -->

File: urdf/gazebo_ros2control.urdf.xacro (robot description, xacro)
@@ -14,5 +14,5 @@
             <state_interface name="position" />
         </joint>
-         <joint name="joint_wheel_right">
+        <joint name="joint_wheel_right">
             <command_interface name="velocity">
                 <param name="min">-10.0</param>
@@ -20,4 +20,15 @@
             </command_interface>
             <state_interface name="velocity" />
+            <state_interface name="position" />
+        </joint>
+        <joint name="caster_roll_joint">
+            <state_interface name="position" />
+            <state_interface name="velocity" />
+        </joint>
+        <joint name="caster_pitch_joint">
+            <state_interface name="position" />
+            <state_interface name="velocity" />
+        </joint>
+        <joint name="caster_mount_joint">
             <state_interface name="position" />
         </joint>
